File: KiCad-Project/Remake-Tank-Mouse.kicad_pcb (KiCad board)
At the start: 2 copper layers, 84.5 x 56.1 mm, 0 parts

Commit message: no message
Parts:
- added Button1: SW_Push_1P1T_NO_6x6mm_H9.5mm, Button_Switch_SMD:SW_Push_1P1T_NO_6x6mm_H9.5mm, F.Cu at (6.82, 40.5)
- added Button2: SW_Push_1P1T_NO_6x6mm_H9.5mm, Button_Switch_SMD:SW_Push_1P1T_NO_6x6mm_H9.5mm, F.Cu at (6.82, 15.5)
Changed lines of the file:
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@@
   (general
     (thickness 1.6)
-    (drawings 10)
+    (drawings 11)
     (tracks 0)
     (zones 0)
-    (modules 0)
+    (modules 2)
     (nets 1)
   )
@@
     (solder_mask_min_width 0.25)
     (aux_axis_origin 0 0)
-    (grid_origin 142.24 93.98)
     (visible_elements FFFFFFFF)
     (pcbplotparams
@@
     (uvia_drill 0.1)
   )
+  (module Button_Switch_SMD:SW_Push_1P1T_NO_6x6mm_H9.5mm (layer F.Cu)
+    (at 6.82 40.535 90)
+    (descr "tactile push button, 6x6mm e.g. PTS645xx series, height=9.5mm")
+    (tags "tact sw push 6mm smd")
+    (attr smd)
+    (fp_text reference Button1 (at 0 -4.05 90) (layer F.SilkS)
+      (effects (font (size 1 1) (thickness 0.15)))
+    )
+    (fp_text value SW_Push_1P1T_NO_6x6mm_H9.5mm (at 0 4.15 90) (layer F.Fab)
+      (effects (font (size 1 1) (thickness 0.15)))
+    )
+    (fp_text user %R (at 0 -4.05 90) (layer F.Fab)
+      (effects (font (size 1 1) (thickness 0.15)))
+    )
+    (fp_line (start -3 -3) (end -3 3) (layer F.Fab) (width 0.1))
+    (fp_line (start -3 3) (end 3 3) (layer F.Fab) (width 0.1))
+    (fp_line (start 3 3) (end 3 -3) (layer F.Fab) (width 0.1))
+    (fp_line (start 3 -3) (end -3 -3) (layer F.Fab) (width 0.1))
+    (fp_line (start 5 3.25) (end 5 -3.25) (layer F.CrtYd) (width 0.05))
+    (fp_line (start -5 -3.25) (end -5 3.25) (layer F.CrtYd) (width 0.05))
+    (fp_line (start -5 3.25) (end 5 3.25) (layer F.CrtYd) (width 0.05))
+    (fp_line (start -5 -3.25) (end 5 -3.25) (layer F.CrtYd) (width 0.05))
+    (fp_line (start 3.23 -3.23) (end 3.23 -3.2) (layer F.SilkS) (width 0.12))
+    (fp_line (start 3.23 3.23) (end 3.23 3.2) (layer F.SilkS) (width 0.12))
+    (fp_line (start -3.23 3.23) (end -3.23 3.2) (layer F.SilkS) (width 0.12))
+    (fp_line (start -3.23 -3.2) (end -3.23 -3.23) (layer F.SilkS) (width 0.12))
+    (fp_line (start 3.23 -1.3) (end 3.23 1.3) (layer F.SilkS) (width 0.12))
+    (fp_line (start -3.23 -3.23) (end 3.23 -3.23) (layer F.SilkS) (width 0.12))
+    (fp_line (start -3.23 -1.3) (end -3.23 1.3) (layer F.SilkS) (width 0.12))
+    (fp_line (start -3.23 3.23) (end 3.23 3.23) (layer F.SilkS) (width 0.12))
+    (fp_circle (center 0 0) (end 1.75 -0.05) (layer F.Fab) (width 0.1))
+    (pad 2 smd rect (at -3.975 2.25 90) (size 1.55 1.3) (layers F.Cu F.Paste F.Mask))
+    (pad 1 smd rect (at -3.975 -2.25 90) (size 1.55 1.3) (layers F.Cu F.Paste F.Mask))
+    (pad 1 smd rect (at 3.975 -2.25 90) (size 1.55 1.3) (layers F.Cu F.Paste F.Mask))
+    (pad 2 smd rect (at 3.975 2.25 90) (size 1.55 1.3) (layers F.Cu F.Paste F.Mask))
+    (model ${KISYS3DMOD}/Button_Switch_SMD.3dshapes/SW_PUSH_6mm_H9.5mm.wrl
+      (at (xyz 0 0 0))
+      (scale (xyz 1 1 1))
+      (rotate (xyz 0 0 0))
+    )
+  )
+  (module Button_Switch_SMD:SW_Push_1P1T_NO_6x6mm_H9.5mm (layer F.Cu)
+    (at 6.82 15.535 90)
+    (descr "tactile push button, 6x6mm e.g. PTS645xx series, height=9.5mm")
+    (tags "tact sw push 6mm smd")
+    (attr smd)
+    (fp_text reference Button2 (at 0 -4.05 90) (layer F.SilkS)
+      (effects (font (size 1 1) (thickness 0.15)))
+    )
+    (fp_text value SW_Push_1P1T_NO_6x6mm_H9.5mm (at 0 4.15 90) (layer F.Fab)
+      (effects (font (size 1 1) (thickness 0.15)))
+    )
+    (fp_circle (center 0 0) (end 1.75 -0.05) (layer F.Fab) (width 0.1))
+    (fp_line (start -3.23 3.23) (end 3.23 3.23) (layer F.SilkS) (width 0.12))
+    (fp_line (start -3.23 -1.3) (end -3.23 1.3) (layer F.SilkS) (width 0.12))
+    (fp_line (start -3.23 -3.23) (end 3.23 -3.23) (layer F.SilkS) (width 0.12))
+    (fp_line (start 3.23 -1.3) (end 3.23 1.3) (layer F.SilkS) (width 0.12))
+    (fp_line (start -3.23 -3.2) (end -3.23 -3.23) (layer F.SilkS) (width 0.12))
+    (fp_line (start -3.23 3.23) (end -3.23 3.2) (layer F.SilkS) (width 0.12))
+    (fp_line (start 3.23 3.23) (end 3.23 3.2) (layer F.SilkS) (width 0.12))
+    (fp_line (start 3.23 -3.23) (end 3.23 -3.2) (layer F.SilkS) (width 0.12))
+    (fp_line (start -5 -3.25) (end 5 -3.25) (layer F.CrtYd) (width 0.05))
+    (fp_line (start -5 3.25) (end 5 3.25) (layer F.CrtYd) (width 0.05))
+    (fp_line (start -5 -3.25) (end -5 3.25) (layer F.CrtYd) (width 0.05))
+    (fp_line (start 5 3.25) (end 5 -3.25) (layer F.CrtYd) (width 0.05))
+    (fp_line (start 3 -3) (end -3 -3) (layer F.Fab) (width 0.1))
+    (fp_line (start 3 3) (end 3 -3) (layer F.Fab) (width 0.1))
+    (fp_line (start -3 3) (end 3 3) (layer F.Fab) (width 0.1))
+    (fp_line (start -3 -3) (end -3 3) (layer F.Fab) (width 0.1))
+    (fp_text user %R (at 0 -4.05 90) (layer F.Fab)
+      (effects (font (size 1 1) (thickness 0.15)))
+    )
+    (pad 2 smd rect (at 3.975 2.25 90) (size 1.55 1.3) (layers F.Cu F.Paste F.Mask))
+    (pad 1 smd rect (at 3.975 -2.25 90) (size 1.55 1.3) (layers F.Cu F.Paste F.Mask))
+    (pad 1 smd rect (at -3.975 -2.25 90) (size 1.55 1.3) (layers F.Cu F.Paste F.Mask))
+    (pad 2 smd rect (at -3.975 2.25 90) (size 1.55 1.3) (layers F.Cu F.Paste F.Mask))
+    (model ${KISYS3DMOD}/Button_Switch_SMD.3dshapes/SW_PUSH_6mm_H9.5mm.wrl
+      (at (xyz 0 0 0))
+      (scale (xyz 1 1 1))
+      (rotate (xyz 0 0 0))
+    )
+  )
+  (gr_line (start 0 28.035) (end 34.5 28.035) (layer F.SilkS) (width 0.12))
   (gr_circle (center 34.5 28.035) (end 34.5 30.285) (layer Edge.Cuts) (width 0.05))
   (gr_circle (center 77.5 28.035) (end 77.5 30.285) (layer Edge.Cuts) (width 0.05))
